Commit message: Add torque values into KR20 and KR16 URDFs

File: kuka_kr16_support/urdf/kr16_2_macro.xacro (robot description, xacro)
@@ -154,5 +154,5 @@
       <child link="${prefix}link_1"/>
       <axis xyz="0 0 -1"/>
-      <limit effort="0" lower="${radians(-185)}" upper="${radians(185)}" velocity="${radians(156)}"/>
+      <limit effort="2500" lower="${radians(-185)}" upper="${radians(185)}" velocity="${radians(156)}"/>
     </joint>
     <!-- joint 2 (A2) -->
@@ -162,5 +162,5 @@
       <child link="${prefix}link_2"/>
       <axis xyz="0 1 0"/>
-      <limit effort="0" lower="${radians(-155)}" upper="${radians(35)}" velocity="${radians(156)}"/>
+      <limit effort="3100" lower="${radians(-155)}" upper="${radians(35)}" velocity="${radians(156)}"/>
     </joint>
     <!-- joint 3 (A3) -->
@@ -170,5 +170,5 @@
       <child link="${prefix}link_3"/>
       <axis xyz="0 1 0"/>
-      <limit effort="0" lower="${radians(-130)}" upper="${radians(154)}" velocity="${radians(156)}"/>
+      <limit effort="2200" lower="${radians(-130)}" upper="${radians(154)}" velocity="${radians(156)}"/>
     </joint>
     <!-- joint 4 (A4) -->
@@ -178,5 +178,5 @@
       <child link="${prefix}link_4"/>
       <axis xyz="-1 0 0"/>
-      <limit effort="0" lower="${radians(-350)}" upper="${radians(350)}" velocity="${radians(330)}"/>
+      <limit effort="500" lower="${radians(-350)}" upper="${radians(350)}" velocity="${radians(330)}"/>
     </joint>
     <!-- joint 5 (A5) -->
@@ -186,5 +186,5 @@
       <child link="${prefix}link_5"/>
       <axis xyz="0 1 0"/>
-      <limit effort="0" lower="${radians(-130)}" upper="${radians(130)}" velocity="${radians(330)}"/>
+      <limit effort="500" lower="${radians(-130)}" upper="${radians(130)}" velocity="${radians(330)}"/>
     </joint>
     <!-- joint 6 (A6) -->
@@ -194,5 +194,5 @@
       <child link="${prefix}link_6"/>
       <axis xyz="-1 0 0"/>
-      <limit effort="0" lower="${radians(-350)}" upper="${radians(350)}" velocity="${radians(615)}"/>
+      <limit effort="150" lower="${radians(-350)}" upper="${radians(350)}" velocity="${radians(615)}"/>
     </joint>
     <!-- tool frame - fixed frame -->

File: kuka_kr20_support/urdf/kr20_r1810_2_macro.xacro (robot description, xacro)
@@ -163,5 +163,5 @@
       <child link="${prefix}link_1"/>
       <axis xyz="0 0 -1"/>
-      <limit effort="0" lower="${radians(-185)}" upper="${radians(185)}" velocity="${radians(200)}"/>
+      <limit effort="2500" lower="${radians(-185)}" upper="${radians(185)}" velocity="${radians(200)}"/>
     </joint>
     <!-- joint 2 (A2) -->
@@ -171,5 +171,5 @@
       <child link="${prefix}link_2"/>
       <axis xyz="0 1 0"/>
-      <limit effort="0" lower="${radians(-185)}" upper="${radians(65)}" velocity="${radians(175)}"/>
+      <limit effort="3100" lower="${radians(-185)}" upper="${radians(65)}" velocity="${radians(175)}"/>
     </joint>
     <!-- joint 3 (A3) -->
@@ -179,5 +179,5 @@
       <child link="${prefix}link_3"/>
       <axis xyz="0 1 0"/>
-      <limit effort="0" lower="${radians(-138)}" upper="${radians(175)}" velocity="${radians(190)}"/>
+      <limit effort="2200" lower="${radians(-138)}" upper="${radians(175)}" velocity="${radians(190)}"/>
     </joint>
     <!-- joint 4 (A4) -->
@@ -187,5 +187,5 @@
       <child link="${prefix}link_4"/>
       <axis xyz="-1 0 0"/>
-      <limit effort="0" lower="${radians(-350)}" upper="${radians(350)}" velocity="${radians(430)}"/>
+      <limit effort="500" lower="${radians(-350)}" upper="${radians(350)}" velocity="${radians(430)}"/>
     </joint>
     <!-- joint 5 (A5) -->
@@ -195,5 +195,5 @@
       <child link="${prefix}link_5"/>
       <axis xyz="0 1 0"/>
-      <limit effort="0" lower="${radians(-130)}" upper="${radians(130)}" velocity="${radians(430)}"/>
+      <limit effort="500" lower="${radians(-130)}" upper="${radians(130)}" velocity="${radians(430)}"/>
     </joint>
     <!-- joint 6 (A6) -->
@@ -203,5 +203,5 @@
       <child link="${prefix}link_6"/>
       <axis xyz="-1 0 0"/>
-      <limit effort="0" lower="${radians(-350)}" upper="${radians(350)}" velocity="${radians(630)}"/>
+      <limit effort="150" lower="${radians(-350)}" upper="${radians(350)}" velocity="${radians(630)}"/>
     </joint>
     <!-- tool frame - fixed frame -->

Commit message: Change limit value KR16

File: kuka_kr16_support/urdf/kr16_2_macro.xacro (robot description, xacro)
@@ -7,5 +7,5 @@
       <inertial>
         <origin xyz="0 0 0" rpy="0 0 0"/>
-        <mass value="2"/>
+        <mass value="2500"/>
         <inertia ixx="0.01" ixy="0" ixz="0" iyy="0.01" iyz="0" izz="0.01" />
       </inertial>
